File: pcb/rgb-pcb.sch (KiCad schematic (older format))
At the start: 13 parts

Commit message: Continued schematic work
Parts:
- added IC?: VCC_REG, symbol VCC_REG
- added J?: SER-POW_IN, symbol SER-POW_IN
- added P?: AVR_ISP, symbol AVR_ISP
- added R? (x2): 10k, symbol R
- added S?: SPST, symbol SPST
Connections:
- net GND: now also IC?.2 (COMMON), J?.3 (GND), J?.4 (GND), P?.6 (GND), S?.1; no longer C?.1, C?.1, IC?.18 (AVCC), IC?.20 (AREF), IC?.28 (VCC), IC?.4 (VCC), IC?.6 (VCC), LED?.4 (R_A), LED?.4 (R_A), LED?.4 (R_A), LED?.4 (R_A), LED?.4 (R_A), LED?.5 (G_A), LED?.5 (G_A), LED?.5 (G_A), LED?.5 (G_A), LED?.5 (G_A), LED?.6 (B_A), LED?.6 (B_A), LED?.6 (B_A), LED?.6 (B_A), LED?.6 (B_A)
- net FEEDBACK: now reaches IC?.1 (PD3(PCINT19/OC2B/INT1))
- net FEEDBACK: now also IC?.24 (SOUT)
- net CLOCK: now reaches IC?.12 (PB0(PCINT0/CLKO/ICP1))
- net CLOCK: now also IC?.25 (GSCLK)
- net BLANK: now reaches IC?.13 (PB1(PCINT1/OC1A))
- net BLANK: now also IC?.2 (BLANK), R?.1
- net LATCH: now reaches IC?.14 (PB2(PCINT2/~SS~/OC1B))
- net LATCH: now also IC?.3 (XLAT)
- net SPI_MOSI: now reaches IC?.15 (PB3(PCINT3/OC2A/MOSI))
- net SPI_MOSI: now also IC?.5 (SIN), P?.4 (MOSI)
- net SPI_MISO: now reaches IC?.16 (PB4(PCINT4/MISO))
- net SPI_MISO: now also P?.1 (MISO)
- net SPI_SCK: now reaches IC?.17 (PB5(SCK/PCINT5))
- net SPI_SCK: now also IC?.4 (SCLK), P?.3 (SCK)
- net DC_MODE: now reaches IC?.2 (PD4(PCINT20/XCK/T0))
- net DC_MODE: now also IC?.25 (GSCLK)
- net RESET: now reaches IC?.29 (~RESET~(PC6))
- net RESET: now also P?.5 (RESET), R?.1, S?.2
- net SER_RX: now reaches IC?.30 (PD0(RXD/PCINT16))
- net SER_TX: now reaches IC?.31 (PD1(TXD/PCINT17))
- net ERROR: now reaches IC?.32 (PD2(INT0/PCINT18))
- net ERROR: now also IC?.23 (XERR)
- net SUPER: now reaches IC?.9 (PD5(PCINT21/OC0B/T1))
- net SUPER: now also IC?.6 (VPRG)
- new net VCC: C?.1, C?.1, IC?.18 (AVCC), IC?.20 (AREF), IC?.28 (VCC), IC?.3 (OUTPUT), IC?.4 (VCC), IC?.6 (VCC), LED?.4 (R_A), LED?.4 (R_A), LED?.4 (R_A), LED?.4 (R_A), LED?.4 (R_A), LED?.5 (G_A), LED?.5 (G_A), LED?.5 (G_A), LED?.5 (G_A), LED?.5 (G_A), LED?.6 (B_A), LED?.6 (B_A), LED?.6 (B_A), LED?.6 (B_A), LED?.6 (B_A), P?.2 (VCC), R?.2, R?.2
- new net V_BUS: IC?.1 (INPUT), J?.1 (VBUS), J?.2 (VBUS)
- no-connect marks 1 -> 3
